File: EMSBoard.sch (EAGLE design)
At the start: 5 parts, among them IC2 BLUE_PILL, J1 B2B-XH-A__LF__SN_

Commit message: Resolve Conflicts
Parts:
- J1: value B2B-XH-A__LF__SN_ -> (none); device SamacSys_Parts:B2B-XH-A__LF__SN_ -> jst-xh:S2B-XH-A
Connections:
- net GND: now also IC2.G$3; no longer IC2.G$1
Other:
- moved on the sheet: J1
Changed lines of the file:
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@@
 <parts>
 <part name="IC2" library="stm32_mcu" deviceset="BLUE_PILL" device=""/>
-<part name="J1" library="SamacSys_Parts" deviceset="B2B-XH-A__LF__SN_" device=""/>
+<part name="J1" library="jst-xh" deviceset="S2B-XH-A" device=""/>
 <part name="D3" library="led" library_urn="urn:adsk.eagle:library:259" deviceset="LED" device="CHIP-LED0805" package3d_urn="urn:adsk.eagle:package:15818/2"/>
 <part name="R2" library="rcl" library_urn="urn:adsk.eagle:library:334" deviceset="R-EU_" device="R0603" package3d_urn="urn:adsk.eagle:package:23555/3" value="1k"/>
@@
 <attribute name="VALUE" x="12.7" y="86.36" size="1.778" layer="96" rot="R180"/>
 </instance>
-<instance part="J1" gate="G$1" x="66.04" y="71.12" smashed="yes">
-<attribute name="NAME" x="82.55" y="78.74" size="1.778" layer="95" align="center-left"/>
-<attribute name="VALUE" x="82.55" y="76.2" size="1.778" layer="96" align="center-left"/>
+<instance part="J1" gate="G$1" x="71.12" y="71.12" smashed="yes">
+<attribute name="NAME" x="72.39" y="76.2" size="1.778" layer="95" align="center-left"/>
+<attribute name="VALUE" x="87.63" y="76.2" size="1.778" layer="96" align="center-left"/>
 </instance>
 <instance part="D3" gate="G$1" x="45.72" y="50.8" smashed="yes">
@@
 <attribute name="VALUE" x="43.18" y="35.56" size="1.778" layer="96"/>
 </instance>
-<instance part="GND2" gate="1" x="40.64" y="78.74" smashed="yes">
-<attribute name="VALUE" x="38.1" y="76.2" size="1.778" layer="96"/>
+<instance part="GND2" gate="1" x="-7.62" y="30.48" smashed="yes">
+<attribute name="VALUE" x="-10.16" y="27.94" size="1.778" layer="96"/>
 </instance>
 </instances>
@@
 <pinref part="R4" gate="G$1" pin="1"/>
 <pinref part="J1" gate="G$1" pin="1"/>
-<wire x1="66.04" y1="71.12" x2="66.04" y2="68.58" width="0.1524" layer="91"/>
-<junction x="66.04" y="68.58"/>
+<wire x1="71.12" y1="71.12" x2="71.12" y2="68.58" width="0.1524" layer="91"/>
+<junction x="71.12" y="68.58"/>
+<wire x1="71.12" y1="68.58" x2="66.04" y2="68.58" width="0.1524" layer="91"/>
 </segment>
 </net>
@@
 <net name="GND" class="0">
 <segment>
-<pinref part="IC2" gate="G$1" pin="G$1"/>
-<pinref part="GND2" gate="1" pin="GND"/>
-<wire x1="27.94" y1="81.28" x2="40.64" y2="81.28" width="0.1524" layer="91"/>
-</segment>
-<segment>
 <pinref part="GND1" gate="1" pin="GND"/>
 <pinref part="D3" gate="G$1" pin="C"/>
 <wire x1="45.72" y1="40.64" x2="45.72" y2="45.72" width="0.1524" layer="91"/>
 </segment>
+<segment>
+<pinref part="IC2" gate="G$1" pin="G$3"/>
+<pinref part="GND2" gate="1" pin="GND"/>
+<wire x1="2.54" y1="35.56" x2="-7.62" y2="35.56" width="0.1524" layer="91"/>
+<wire x1="-7.62" y1="35.56" x2="-7.62" y2="33.02" width="0.1524" layer="91"/>
+</segment>
 </net>

Commit message: Solid Ground
Connections:
- net GND: now also IC2.G$0, IC2.G$1
Changed lines of the file:
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@@
 <part name="GND1" library="supply1" library_urn="urn:adsk.eagle:library:371" deviceset="GND" device=""/>
 <part name="GND2" library="supply1" library_urn="urn:adsk.eagle:library:371" deviceset="GND" device=""/>
+<part name="GND3" library="supply1" library_urn="urn:adsk.eagle:library:371" deviceset="GND" device=""/>
 </parts>
 <sheets>
@@
 <instance part="GND2" gate="1" x="-7.62" y="30.48" smashed="yes">
 <attribute name="VALUE" x="-10.16" y="27.94" size="1.778" layer="96"/>
+</instance>
+<instance part="GND3" gate="1" x="35.56" y="73.66" smashed="yes">
+<attribute name="VALUE" x="33.02" y="71.12" size="1.778" layer="96"/>
 </instance>
 </instances>
@@
 <wire x1="-7.62" y1="35.56" x2="-7.62" y2="33.02" width="0.1524" layer="91"/>
 </segment>
+<segment>
+<pinref part="IC2" gate="G$1" pin="G$1"/>
+<pinref part="GND3" gate="1" pin="GND"/>
+<wire x1="27.94" y1="81.28" x2="35.56" y2="81.28" width="0.1524" layer="91"/>
+<wire x1="35.56" y1="81.28" x2="35.56" y2="78.74" width="0.1524" layer="91"/>
+<pinref part="IC2" gate="G$1" pin="G$0"/>
+<wire x1="35.56" y1="78.74" x2="35.56" y2="76.2" width="0.1524" layer="91"/>
+<wire x1="27.94" y1="78.74" x2="35.56" y2="78.74" width="0.1524" layer="91"/>
+<junction x="35.56" y="78.74"/>
+</segment>
 </net>
